Commit message: added camera, imu sensors

File: robot_descriptions/urdf/common_parameters.xacro (robot description, xacro)
@@ -13,29 +13,29 @@
         <color rgba="1.0 1.0 0 1" />
     </material>
-    <xacro:macro name="box_inertia" params="m l w h xyz rpy">
+    <xacro:macro name="box_inertia" params="mass length width height xyz rpy">
         <inertial>
             <origin xyz="${xyz}" rpy="${rpy}" />
-            <mass value="${m}" />
-            <inertia ixx="${(m/12) * (h*h + l*l)}" ixy="0" ixz="0"
-                     iyy="${(m/12) * (w*w + l*l)}" iyz="0"
-                     izz="${(m/12) * (w*w + h*h)}" />
+            <mass value="${mass}" />
+            <inertia ixx="${(mass/12) * (height * height + length * length)}" ixy="0" ixz="0"
+                     iyy="${(mass/12) * (width * width + length * length)}" iyz="0"
+                     izz="${(mass/12) * (width * width + height * height)}" />
         </inertial>
     </xacro:macro>
-    <xacro:macro name="cylinder_inertia" params="m r h xyz rpy">
+    <xacro:macro name="cylinder_inertia" params="mass radius height xyz rpy">
         <inertial>
             <origin xyz="${xyz}" rpy="${rpy}" />
-            <mass value="${m}" />
-            <inertia ixx="${(m/12) * (3*r*r + h*h)}" ixy="0" ixz="0"
-                     iyy="${(m/12) * (3*r*r + h*h)}" iyz="0"
-                     izz="${(m/2) * (r*r)}" />
+            <mass value="${mass}" />
+            <inertia ixx="${(mass/12) * (3 * radius * radius + height * height)}" ixy="0" ixz="0"
+                     iyy="${(mass/12) * (3 * radius * radius + height * height)}" iyz="0"
+                     izz="${(mass/2) * (radius * radius)}" />
         </inertial>
     </xacro:macro>
-    <xacro:macro name="sphere_inertia" params="m r xyz rpy">
+    <xacro:macro name="sphere_inertia" params="mass radius xyz rpy">
         <inertial>
             <origin xyz="${xyz}" rpy="${rpy}" />
-            <mass value="${m}" />
-            <inertia ixx="${(2/5) * m * r * r}" ixy="0" ixz="0"
-                     iyy="${(2/5) * m * r * r}" iyz="0"
-                     izz="${(2/5) * m * r * r}" />
+            <mass value="${mass}" />
+            <inertia ixx="${(2/5) * mass * radius * radius}" ixy="0" ixz="0"
+                     iyy="${(2/5) * mass * radius * radius}" iyz="0"
+                     izz="${(2/5) * mass * radius * radius}" />
         </inertial>
     </xacro:macro>

File: robot_descriptions/urdf/vanilla_bot/vanilla_bot_base.xacro (robot description, xacro)
@@ -2,16 +2,22 @@
 <robot xmlns:xacro="http://www.ros.org/wiki/xacro">
     <!-- Parameters for mobile base -->
-    <xacro:property name="base_length" value ="0.07"/>
+    <xacro:property name="base_length" value ="0.1"/>
     <xacro:property name="base_radius" value ="0.8"/>
-    <!-- Parametesr for mobile base wheels -->
+    <!-- Parameters for mobile base wheels -->
     <xacro:property name="wheel_radius" value ="0.18"/>
     <xacro:property name="wheel_length" value ="0.05"/>
-    <!-- Parametesr for mobile base caster wheels -->
+    <!-- Parameters for mobile base caster wheels -->
     <xacro:property name="caster_wheel_radius" value ="0.07"/>
     <xacro:property name="caster_wheel_length" value ="${((base_length / 2) * 2)+(wheel_radius)}"/>
-    <xacro:property name="lider" value ="0.15"/>
-    <xacro:property name="camera_length" value="0.01" />
-    <xacro:property name="camera_width" value="0.05" />
-    <xacro:property name="camera_hight" value="0.1" />
+    <!--  Parameters for IMU -->
+    <xacro:imu  link_name = "imu_link" parent_link = "base_link" joint_name = "imu_joint"
+                xyz="0.0 0.0 ${base_length/2}" rpy="0.0 0.0 0.0" />
+    <!--  Parameters for Camera -->
+    <xacro:camera link_name = "camera_link" parent_link = "base_link" joint_name = "camera_joint"
+                  camera_length = "0.02" camera_width = "0.1" camera_height = "${base_length}" mass = "0.01"
+                  Vxyz = "0 0 0" Vrpy = "0 0 0" Jxyz = "${base_radius} 0 ${base_length/2}" Jrpy = "0 0 0"
+                  />
+<!--  Parameters for Laser Sensor -->
+    <!-- <xacro:property name="lider" value ="0.15"/> -->
 <!-- ********************** Base footprint link and joint ********************** -->
     <link name="base_footprint"/>
@@ -35,7 +41,10 @@
             </geometry>
         </collision>
-        <xacro:cylinder_inertia m="1.0" r="${base_radius}" h="${base_length}"
+        <xacro:cylinder_inertia mass="1.0" radius="${base_radius}" height="${base_length}"
                                     xyz="0 0 ${base_length/2}" rpy="0 0 ${pi / 2.0}" />
     </link>
+    <gazebo reference="base_link">
+        <material>Gazebo/Blue</material>
+    </gazebo>
 <!-- ********************** Wheel links and joints ********************** -->
     <xacro:macro name="wheel_link" params="prefix">
@@ -54,5 +63,5 @@
                 </geometry>
             </collision>
-            <xacro:cylinder_inertia m="0.05" r="${wheel_radius}" h="${wheel_length}"
+            <xacro:cylinder_inertia mass="0.05" radius="${wheel_radius}" height="${wheel_length}"
                                     xyz="0 0 0" rpy="${pi / 2.0} 0 0" />
         </link>
@@ -61,5 +70,6 @@
     <xacro:wheel_link prefix="left" />
     <joint name="base_right_wheel_joint" type="continuous">
-        <origin xyz="0.0 ${(base_radius)+(wheel_length / 2)} ${-((base_length / 2) * 2)}" rpy="0.0 0.0 0.0"/>
+        <origin xyz="0.0 ${(base_radius)+(wheel_length / 2)} ${-((base_length / 2) * 2)}"
+                rpy="0.0 0.0 0.0"/>
         <parent link="base_link"/>
         <child link="right_wheel_link"/>
@@ -67,14 +77,22 @@
     </joint>
     <joint name="base_left_wheel_joint" type="continuous">
-        <origin xyz="0.0 ${-((base_radius)+(wheel_length / 2))} ${-((base_length / 2) * 2)}" rpy="0.0 0.0 0.0"/>
+        <origin xyz="0.0 ${-((base_radius)+(wheel_length / 2))} ${-((base_length / 2) * 2)}"
+                rpy="0.0 0.0 0.0"/>
         <parent link="base_link"/>
         <child link="left_wheel_link"/>
         <axis xyz="0.0 1 0.0"/>
     </joint>
+    <gazebo reference="right_wheel_link">
+        <material>Gazebo/Grey</material>
+    </gazebo>
+    <gazebo reference="left_wheel_link">
+        <material>Gazebo/Grey</material>
+    </gazebo>
 <!-- ********************** caster wheel links and joints ********************** -->
     <xacro:macro name="caster_wheel_link" params="prefix">
         <link name="${prefix}_caster_wheel_link">
             <visual name="caster_wheel_handel">
-                <origin xyz="0.0 0.0 ${-((caster_wheel_length-caster_wheel_radius)/2)}" rpy="0.0 0.0 0.0"/>
+                <origin xyz="0.0 0.0 ${-((caster_wheel_length-caster_wheel_radius)/2)}"
+                        rpy="0.0 0.0 0.0"/>
                 <geometry>
                     <cylinder radius="${caster_wheel_radius}" length="${caster_wheel_length - caster_wheel_radius}"/>
@@ -82,5 +100,6 @@
             </visual>
             <visual name="caster_wheel">
-                <origin xyz="0.0 0.0 ${-((caster_wheel_length/2)*2)+caster_wheel_radius}" rpy="0.0 0.0 0.0"/>
+                <origin xyz="0.0 0.0 ${-((caster_wheel_length/2)*2)+caster_wheel_radius}"
+                        rpy="0.0 0.0 0.0"/>
                 <geometry>
                     <sphere radius="${caster_wheel_radius}"/>
@@ -93,6 +112,7 @@
                 </geometry>
             </collision>
-            <xacro:cylinder_inertia m="0.04" r="${caster_wheel_radius}" h="${caster_wheel_length}"
-                                    xyz="0 0 ${-((caster_wheel_length-caster_wheel_radius)/2)}" rpy="0 0 0" />
+            <xacro:cylinder_inertia mass="0.04" radius="${caster_wheel_radius}" height="${caster_wheel_length}"
+                                    xyz="0 0 ${-((caster_wheel_length-caster_wheel_radius)/2)}"
+                                    rpy="0 0 0" />
         </link>
     </xacro:macro>
@@ -109,55 +129,13 @@
         <child link="back_caster_wheel_link"/>
     </joint>
-<!-- ********************** Imu links and joints ********************** -->
-    <link name="imu_link"/>
-    <joint name="base_imu_joint" type="fixed">
-        <origin xyz="0.0 0.0 ${base_length/2}" rpy="0.0 0.0 0.0"/>
-        <parent link="base_link"/>
-        <child link="imu_link"/>
-    </joint>
-<!-- ********************** Lider links and joints ********************** -->
-    <link name="lider_link">
-        <visual name="">
-            <origin xyz="0.0 0.0 ${lider/2}" rpy="0.0 0.0 0.0"/>
-            <geometry>
-                <box size="${lider} ${lider} ${lider}"/>
-            </geometry>
-        </visual>
-        <collision>
-            <origin xyz="0.0 0.0 ${lider/2}" rpy="0.0 0.0 0.0"/>
-            <geometry>
-                <box size="${lider} ${lider} ${lider}"/>
-            </geometry>
-        </collision>
-        <xacro:box_inertia m="0.1" l="${lider}" w="${lider}" h="${lider}"
-                           xyz="0 0 0" rpy="0 0 0" />
-    </link>
-    <joint name="base_lider_joint" type="fixed">
-        <origin xyz="0.0 0.0 ${base_length}" rpy="0.0 0.0 0.0"/>
-        <parent link="base_link"/>
-        <child link="lider_link"/>
-    </joint>
-<!-- ********************** Camera links and joints ********************** -->
-    <link name="camera_link">
-        <visual>
-            <origin xyz="0.0 0.0 ${-(camera_hight-0.05)}" rpy="0.0 0.0 0.0"/>
-            <geometry>
-                <box size="${camera_length} ${camera_width} ${camera_hight}"/>
-            </geometry>
-            <material name="grey"/>
-        </visual>
-        <collision>
-            <origin xyz="0.0 0.0 ${-(camera_hight-0.05)}" rpy="0.0 0.0 0.0"/>
-            <geometry>
-                <box size="${camera_length} ${camera_width} ${camera_hight}"/>
-            </geometry>
-        </collision>
-        <xacro:box_inertia m="0.1" l="${camera_length}" w="${camera_width}" h="${camera_hight}"
-                           xyz="0 0 0" rpy="0 0 0" />
-    </link>
-    <joint name="base_camera_joint" type="fixed">
-        <origin xyz="${lider/2} 0.0 ${base_length + lider+(camera_hight)}" rpy="0.0 0.0 0.0"/>
-        <parent link="base_link"/>
-        <child link="camera_link"/>
-    </joint>
+    <gazebo reference="front_caster_wheel_link">
+        <material>Gazebo/Grey</material>
+        <mu1 value="0.1" />
+        <mu2 value="0.1" />
+    </gazebo>
+    <gazebo reference="back_caster_wheel_link">
+        <material>Gazebo/Grey</material>
+        <mu1 value="0.1" />
+        <mu2 value="0.1" />
+    </gazebo>
 </robot>

File: robot_descriptions/urdf/vanilla_bot/vanilla_bot_gazebo.xacro (robot description, xacro)
@@ -1,50 +1,76 @@
 <?xml version="1.0"?>
 <robot xmlns:xacro="http://www.ros.org/wiki/xacro">
-    <gazebo reference="base_link">
-        <material>Gazebo/Blue</material>
-    </gazebo>
-    <gazebo reference="right_wheel_link">
-        <material>Gazebo/Grey</material>
-    </gazebo>
-    <gazebo reference="left_wheel_link">
-        <material>Gazebo/Grey</material>
-    </gazebo>
-    <gazebo reference="front_caster_wheel_link">
-        <material>Gazebo/Grey</material>
-        <mu1 value="0.1" />
-        <mu2 value="0.1" />
-    </gazebo>
-    <gazebo reference="back_caster_wheel_link">
-        <material>Gazebo/Grey</material>
-        <mu1 value="0.1" />
-        <mu2 value="0.1" />
-    </gazebo>
     <gazebo>
         <plugin name="diff_drive_controller" filename="libgazebo_ros_diff_drive.so">
-            <!-- Update rate in Hz -->
-            <update_rate>50</update_rate>
-            <!-- wheels -->
-            <right_joint>base_right_wheel_joint</right_joint>
-            <left_joint>base_left_wheel_joint</left_joint>
-            <!-- kinematics -->
-            <wheel_separation>0.825</wheel_separation>
-            <wheel_diameter>0.36</wheel_diameter>
-            <!-- <publish_odom>true</publish_odom> -->
-            <publish_odom_tf>true</publish_odom_tf>
-            <publish_wheel_tf>true</publish_wheel_tf>
-            <odometry_topic>odom</odometry_topic>
-            <odometry_frame>odom</odometry_frame>
-            <robot_base_frame>base_footprint</robot_base_frame>
+        <ros>
+            <!-- <namespace>/br</namespace> -->
+        </ros>
+        <update_rate>50</update_rate>
+        <!-- wheels -->
+        <left_joint>base_left_wheel_joint</left_joint>
+        <right_joint>base_right_wheel_joint</right_joint>
+                <!-- <wheel_separation>0.825</wheel_separation>
+                <wheel_diameter>0.36</wheel_diameter> -->
+        <!-- kinematics -->
+        <wheel_separation>${base_radius + wheel_length}</wheel_separation>
+        <wheel_diameter>${2*wheel_radius}</wheel_diameter>
+        <!-- limits -->
+        <max_wheel_torque>20</max_wheel_torque>
+        <max_wheel_acceleration>1.0</max_wheel_acceleration>
+        <command_topic>cmd_vel</command_topic>
+        <!-- output -->
+        <publish_odom>true</publish_odom>
+        <publish_odom_tf>true</publish_odom_tf>
+        <publish_wheel_tf>false</publish_wheel_tf>
+        <odometry_topic>odom</odometry_topic>
+        <odometry_frame>odom</odometry_frame>
+        <robot_base_frame>base_footprint</robot_base_frame>
         </plugin>
     </gazebo>
-    <gazebo reference="camera_link">
-        <sensor name="camera_sensor" type="camera">
-            <pose>0 0 0 0 0 0</pose>
-            <visualize>true</visualize>
-            <update_rate>10.0</update_rate>
-            <plugin name="camera_controller" filename="libgazebo_ros_camera.so">
-                <frame_name>camera_link</frame_name>
-            </plugin>
-        </sensor>
-    </gazebo>
+<!--     <gazebo reference="camera_link">
+    <sensor type="camera" name="camera_sensor">
+        <always_on>true</always_on>
+        <update_rate>15.0</update_rate>
+        <camera name="camera_sensor">
+            <horizontal_fov>1.46608</horizontal_fov>
+            <image>
+                <width>320</width>
+                <height>180</height>
+                <format>R8G8B8</format>
+            </image>
+            <distortion>
+                <k1>0.0</k1>
+                <k2>0.0</k2>
+                <k3>0.0</k3>
+                <p1>0.0</p1>
+                <p2>0.0</p2>
+                <center>0.5 0.5</center>
+            </distortion>
+        </camera>
+        <plugin name="camera_controller" filename="libgazebo_ros_camera.so">
+            <ros>
+                <!- <namespace>stereo</namespace> ->
+                <remapping>~/image_raw:=image_raw</remapping>
+                <remapping>~/camera_info:=camera_info</remapping>
+            </ros>
+            <!- Set camera name. If empty, defaults to sensor name (i.e. "sensor_name") ->
+            <camera_name>camera_sensor</camera_name>
+            <!- Set TF frame name. If empty, defaults to link name (i.e. "link_name") ->
+            <frame_name>camera_link</frame_name>
+            <hack_baseline>0.2</hack_baseline>
+        </plugin>
+    </sensor>
+    <material>Gazebo/Green</material>
+</gazebo> -->
+    <gazebo>
+    <plugin name="bytes_joint_state" filename="libgazebo_ros_joint_state_publisher.so">
+      <ros>
+        <!-- <namespace>/br</namespace> -->
+        <remapping>~/out:=joint_states</remapping>
+      </ros>
+      <update_rate>30</update_rate>
+      <joint_name>base_left_wheel_joint</joint_name>
+      <joint_name>base_right_wheel_joint</joint_name>
+    </plugin>
+</gazebo>
 </robot>

File: robot_descriptions/urdf/vanilla_bot/vanilla_bot_urdf.xacro (robot description, xacro)
@@ -2,5 +2,7 @@
 <robot name="vanilla_bot" xmlns:xacro="http://www.ros.org/wiki/xacro">
     <xacro:include filename="$(find robot_descriptions)/urdf/common_parameters.xacro" />
+    <xacro:include filename="$(find robot_descriptions)/urdf/sensors/imu.xacro" />
+    <xacro:include filename="$(find robot_descriptions)/urdf/sensors/camera.xacro" />
     <xacro:include filename="vanilla_bot_base.xacro" />
-    <xacro:include filename="vanilla_bot_gazebo.xacro" />
+    <!-- <xacro:include filename="vanilla_bot_gazebo.xacro" />  -->
 </robot>
