Commit message: urdf

File: robot_descriptions/urdf/common_parameters.xacro (robot description, xacro)
@@ -1,15 +1,21 @@
 <?xml version="1.0"?>
 <robot xmlns:xacro="http://www.ros.org/wiki/xacro">
-    <material name="blue">
-        <color rgba="0 0 0.5 1" />
+    <material name="Blue">
+        <color rgba="0.0 0.0 0.5 1" />
     </material>
-    <material name="grey">
+    <material name="Grey">
         <color rgba="0.5 0.5 0.5 1" />
     </material>
-    <material name="orange">
-        <color rgba="1.0 0.5 0 1" />
+    <material name="Orange">
+        <color rgba="1.0 0.5 0.0 1" />
     </material>
-    <material name="yellow">
-        <color rgba="1.0 1.0 0 1" />
+    <material name="Yellow">
+        <color rgba="1.0 1.0 0.0 1" />
+    </material>
+    <material name="Red">
+        <color rgba="1.0 0.0 0.0 1" />
+    </material>
+    <material name="Black">
+        <color rgba="0.0 0.0 0.0 1" />
     </material>
     <xacro:macro name="box_inertia" params="mass length width height xyz rpy">

File: robot_descriptions/urdf/sensors/camera.xacro (robot description, xacro)
@@ -2,10 +2,9 @@
 <robot xmlns:xacro="http://www.ros.org/wiki/xacro">
     <xacro:macro name="camera" params=" link_name parent_link joint_name
-                                        Vxyz Vrpy
                                         camera_length camera_width camera_height mass
-                                        Jxyz Jrpy">
+                                        xyz rpy">
         <link name="${link_name}">
             <visual>
-                <origin xyz="${Vxyz}" rpy="${Vrpy}"/>
+                <origin xyz="0 0 0" rpy="0 0 0"/>
                 <geometry>
                     <box size="${camera_length} ${camera_width} ${camera_height}"/>
@@ -14,5 +13,5 @@
             </visual>
             <collision>
-                <origin xyz="${Vxyz}" rpy="${Vrpy}"/>
+                <origin xyz="0 0 0" rpy="0 0 0"/>
                 <geometry>
                     <box size="${camera_length} ${camera_width} ${camera_height}"/>
@@ -23,5 +22,5 @@
         </link>
         <joint name="${joint_name}" type="fixed">
-            <origin xyz="${Jxyz}" rpy="${Jrpy}"/>
+            <origin xyz="${xyz}" rpy="${rpy}"/>
             <parent link="${parent_link}"/>
             <child link="${link_name}"/>
@@ -29,5 +28,5 @@
         <gazebo reference="${link_name}">
             <material>Gazebo/Red</material>
-            <sensor name="camera" type="camera">
+            <sensor name="camera_sensor" type="camera">
                 <pose> 0 0 0 0 0 0 </pose>
                 <visualize>true</visualize>

File: robot_descriptions/urdf/sensors/laser.xacro (robot description, xacro)
@@ -1,10 +1,10 @@
 <?xml version="1.0"?>
 <robot xmlns:xacro="http://www.ros.org/wiki/xacro" >
-<xacro:macro name="camera" params=" link_name parent_link joint_name
-                                        Vxyz Vrpy
+    <xacro:macro name="laser" params=" link_name parent_link joint_name
                                         laser_length laser_radius mass
-                                        Jxyz Jrpy">
+                                        xyz rpy">
         <link name="${link_name}">
             <visual>
+                <origin xyz="0 0 ${-laser_length/2}" rpy="0 0 0"/>
                 <geometry>
                     <cylinder radius="${laser_radius}" length="${laser_length}"/>
@@ -13,21 +13,21 @@
             </visual>
             <collision>
+                <origin xyz="0 0 ${-laser_length/2}" rpy="0 0 0"/>
                 <geometry>
                     <cylinder radius="${laser_radius}" length="${laser_length}"/>
                 </geometry>
             </collision>
-            <xacro:inertial_cylinder mass="0.1" length="${laser_length}" radius="${laser_radius}">
-                <origin xyz="0 0 0" rpy="0 0 0"/>
-            </xacro:inertial_cylinder>
+            <xacro:cylinder_inertia mass="${mass}" height="${laser_length}" radius="${laser_radius}"
+                                    xyz="0 0 0" rpy="0 0 0" />
         </link>
-        <joint name="laser_joint" type="fixed">
-            <origin xyz="0.25 0 0.1" rpy="0 0 0"/>
-            <parent link="chassis"/>
+        <joint name="${joint_name}" type="fixed">
+            <origin xyz="${xyz}" rpy="${rpy}"/>
+            <parent link="${parent_link}"/>
             <child link="${link_name}"/>
         </joint>
         <gazebo reference="${link_name}">
             <material>Gazebo/Red</material>
-            <sensor name="laser" type="ray">
-                <pose> 0 0 0 0 0 0 </pose>
+            <sensor name="laser_sensor" type="ray">
+                <pose> 1 0 0 0 0 0 </pose>
                 <visualize>true</visualize>
                 <update_rate>10</update_rate>
@@ -42,11 +42,11 @@
                     <range>
                         <min>0.3</min>
-                        <max>12</max>
+                        <max>5</max>
                     </range>
                 </ray>
                 <plugin name="laser_controller" filename="libgazebo_ros_ray_sensor.so">
-                    <ros>
+                    <!-- <ros>
                         <argument>~/out:=scan</argument>
-                    </ros>
+                    </ros> -->
                     <output_type>sensor_msgs/LaserScan</output_type>
                     <frame_name>${link_name}</frame_name>

File: robot_descriptions/urdf/vanilla_bot/vanilla_bot_base.xacro (robot description, xacro)
@@ -16,8 +16,9 @@
     <xacro:camera link_name = "camera_link" parent_link = "base_link" joint_name = "camera_joint"
                   camera_length = "0.02" camera_width = "0.1" camera_height = "${base_length}" mass = "0.01"
-                  Vxyz = "0 0 0" Vrpy = "0 0 0" Jxyz = "${base_radius} 0 ${base_length/2}" Jrpy = "0 0 0"
-                  />
-<!--  Parameters for Laser Sensor -->
-    <!-- <xacro:property name="lider" value ="0.15"/> -->
+                  xyz = "${base_radius} 0 ${base_length/2}" rpy = "0 0 0" />
+    <!--  Parameters for Laser Sensor -->
+    <xacro:laser link_name = "laser_link" parent_link = "base_link" joint_name = "laser_joint"
+                  laser_radius = "0.05" laser_length = "0.1" mass = "0.01"
+                  xyz = "0 0 ${base_length + 0.1}" rpy = "0 0 0" /> <!-- Add laser_length to the xyz in int like 0.1 -->
 <!-- ********************** Base footprint link and joint ********************** -->
     <link name="base_footprint"/>
@@ -34,4 +35,5 @@
                 <cylinder radius="${base_radius}" length="${base_length}"/>
             </geometry>
+            <material name="Blue"/>
         </visual>
         <collision>

File: robot_descriptions/urdf/vanilla_bot/vanilla_bot_urdf.xacro (robot description, xacro)
@@ -4,4 +4,5 @@
     <xacro:include filename="$(find robot_descriptions)/urdf/sensors/imu.xacro" />
     <xacro:include filename="$(find robot_descriptions)/urdf/sensors/camera.xacro" />
+    <xacro:include filename="$(find robot_descriptions)/urdf/sensors/laser.xacro" />
     <xacro:include filename="vanilla_bot_base.xacro" />
     <!-- <xacro:include filename="vanilla_bot_gazebo.xacro" />  -->
