Commit message: Diff_drive added

File: robot_descriptions/urdf/plugins/camera.xacro (robot description, xacro)
@@ -10,5 +10,5 @@
                     <box size="${camera_length} ${camera_width} ${camera_height}"/>
                 </geometry>
-                <material name="grey"/>
+                <material name="Black"/>
             </visual>
             <collision>
@@ -27,5 +27,5 @@
         </joint>
         <gazebo reference="${link_name}">
-            <material>Gazebo/Red</material>
+            <material>Gazebo/Black</material>
             <sensor name="camera_sensor" type="camera">
                 <pose> 0 0 0 0 0 0 </pose>

File: robot_descriptions/urdf/plugins/imu.xacro (robot description, xacro)
@@ -10,5 +10,5 @@
         </joint>
         <gazebo reference="imu_link">
-            <sensor name="br_imu" type="imu">
+            <sensor name="imu_sensor" type="imu">
                 <always_on>true</always_on>
                 <update_rate>100</update_rate>
@@ -58,5 +58,5 @@
                     <ros>
                         <namespace>${link_name}</namespace>
-                        <remapping>~/out:=data</remapping>
+                        <!-- <remapping>~/out:=data</remapping> -->
                     </ros>
                     <initial_orientation_as_reference>false</initial_orientation_as_reference>

File: robot_descriptions/urdf/plugins/laser.xacro (robot description, xacro)
@@ -10,5 +10,5 @@
                     <cylinder radius="${laser_radius}" length="${laser_length}"/>
                 </geometry>
-                <material name="red"/>
+                <material name="Red"/>
             </visual>
             <collision>

File: robot_descriptions/urdf/vanilla_bot/vanilla_bot_base.xacro (robot description, xacro)
@@ -21,4 +21,7 @@
                   laser_radius = "0.05" laser_length = "0.1" mass = "0.01"
                   xyz = "0 0 ${base_length + 0.1}" rpy = "0 0 0" /> <!-- Add laser_length to the xyz in int like 0.1 -->
+    <!-- Parameters for Diff_drive Plugin -->
+    <xacro:diff_drive left_joint_name = "base_left_wheel_joint" right_joint_name = "base_right_wheel_joint" robot_base_frame = "base_footprint"
+                                        wheel_diameter = "${wheel_radius*2}" wheel_separation = "${base_radius*2}" />
 <!-- ********************** Base footprint link and joint ********************** -->
     <link name="base_footprint"/>
@@ -57,5 +60,5 @@
                     <cylinder radius="${wheel_radius}" length="${wheel_length}"/>
                 </geometry>
-                <material name="grey" />
+                <material name="Grey" />
             </visual>
             <collision>
@@ -69,6 +72,6 @@
         </link>
     </xacro:macro>
+    <!-- Right  -->
     <xacro:wheel_link prefix="right" />
-    <xacro:wheel_link prefix="left" />
     <joint name="base_right_wheel_joint" type="continuous">
         <origin xyz="0.0 ${(base_radius)+(wheel_length / 2)} ${-((base_length / 2) * 2)}"
@@ -78,4 +81,9 @@
         <axis xyz="0.0 1 0.0"/>
     </joint>
+    <gazebo reference="right_wheel_link">
+        <material>Gazebo/Grey</material>
+    </gazebo>
+    <!-- Left -->
+    <xacro:wheel_link prefix="left" />
     <joint name="base_left_wheel_joint" type="continuous">
         <origin xyz="0.0 ${-((base_radius)+(wheel_length / 2))} ${-((base_length / 2) * 2)}"
@@ -85,7 +93,4 @@
         <axis xyz="0.0 1 0.0"/>
     </joint>
-    <gazebo reference="right_wheel_link">
-        <material>Gazebo/Grey</material>
-    </gazebo>
     <gazebo reference="left_wheel_link">
         <material>Gazebo/Grey</material>
@@ -119,15 +124,10 @@
         </link>
     </xacro:macro>
+    <!-- Front -->
     <xacro:caster_wheel_link prefix="front" />
-    <xacro:caster_wheel_link prefix="back" />
     <joint name="front_caster_wheel_joint" type="fixed">
         <origin xyz="${base_radius-0.1} 0.0 0.0" rpy="0.0 0.0 0.0"/>
         <parent link="base_link"/>
         <child link="front_caster_wheel_link"/>
-    </joint>
-    <joint name="back_caster_wheel_joint" type="fixed">
-        <origin xyz="${-(base_radius-0.1)} 0.0 0.0" rpy="0.0 0.0 0.0"/>
-        <parent link="base_link"/>
-        <child link="back_caster_wheel_link"/>
     </joint>
     <gazebo reference="front_caster_wheel_link">
@@ -136,4 +136,11 @@
         <mu2 value="0.1" />
     </gazebo>
+    <!-- Back -->
+    <xacro:caster_wheel_link prefix="back" />
+    <joint name="back_caster_wheel_joint" type="fixed">
+        <origin xyz="${-(base_radius-0.1)} 0.0 0.0" rpy="0.0 0.0 0.0"/>
+        <parent link="base_link"/>
+        <child link="back_caster_wheel_link"/>
+    </joint>
     <gazebo reference="back_caster_wheel_link">
         <material>Gazebo/Grey</material>

File: robot_descriptions/urdf/vanilla_bot/vanilla_bot_urdf.xacro (robot description, xacro)
@@ -2,7 +2,8 @@
 <robot name="vanilla_bot" xmlns:xacro="http://www.ros.org/wiki/xacro">
     <xacro:include filename="$(find robot_descriptions)/urdf/common_parameters.xacro" />
-    <xacro:include filename="$(find robot_descriptions)/urdf/sensors/imu.xacro" />
-    <xacro:include filename="$(find robot_descriptions)/urdf/sensors/camera.xacro" />
-    <xacro:include filename="$(find robot_descriptions)/urdf/sensors/laser.xacro" />
+    <xacro:include filename="$(find robot_descriptions)/urdf/plugins/imu.xacro" />
+    <xacro:include filename="$(find robot_descriptions)/urdf/plugins/camera.xacro" />
+    <xacro:include filename="$(find robot_descriptions)/urdf/plugins/laser.xacro" />
+    <xacro:include filename="$(find robot_descriptions)/urdf/plugins/diff_drive.xacro" />
     <xacro:include filename="vanilla_bot_base.xacro" />
     <!-- <xacro:include filename="vanilla_bot_gazebo.xacro" />  -->
