Commit message: readme

File: robot_descriptions/urdf/chocolate_bot/chocolate_bot_base.xacro (robot description, xacro)
@@ -25,10 +25,12 @@
             <material name="Blue"/>
         </visual>
-        <!-- <collision>
+        <collision>
             <origin xyz="0.0 0.0 0" rpy="0.0 0.0 0.0"/>
             <geometry>
-                <box size="0.0 0.0 0.0"/>
+                <box size="0.15 0.10 0.06"/>
             </geometry>
-        </collision> -->
+        </collision>
+        <xacro:box_inertia mass="1.5" length="0.15" width="0.10" height="0.06"
+                            xyz="0 0 0" rpy="0 0 0" />
     </link>
     <gazebo reference="base_link">
@@ -52,10 +54,9 @@
                 <material name="Black" />
             </visual>
-            <!-- <collision>
+            <collision>
                 <origin xyz="0 0 0" rpy="0 0 0" />
                 <geometry>
-                    <mesh filename="file:///$(find robot_descriptions)/urdf/chocolate_bot/meshes/wheel_rim.dae"  scale="10 10 10"/>
                 </geometry>
-            </collision> -->
+            </collision>
             <!-- <xacro:cylinder_inertia mass="0.05" radius="${wheel_radius}" height="${wheel_length}"
                                     xyz="0 0 0" rpy="${pi / 2.0} 0 0" /> -->

Commit message: added skid_drive

File: robot_descriptions/urdf/chocolate_bot/chocolate_bot_base.xacro (robot description, xacro)
@@ -1,16 +1,11 @@
 <?xml version="1.0"?>
 <robot xmlns:xacro="http://www.ros.org/wiki/xacro">
-    <!-- Parameters for mobile base -->
-    <!-- <xacro:property name="base_length" value ="1"/>
-    <xacro:property name="base_width" value ="0.5"/>
-    <xacro:property name="base_height" value ="0.02"/> -->
-    <!-- Parameters for mobile base wheels -->
-    <!-- <xacro:property name="wheel_radius" value ="0.18"/>
-    <xacro:property name="wheel_length" value ="0.05"/>
- -->
+    <xacro:skid_steer_drive leftFrontJoint = "base_front_left_wheel_joint" rightFrontJoint = "base_front_right_wheel_joint"
+                            leftRearJoint = "base_back_left_wheel_joint" rightRearJoint = "base_back_right_wheel_joint"
+                            robotBaseFrame = "base_link" wheelDiameter = "0.165" wheelSeparation = "1" />
 <!-- ********************** Base footprint link and joint ********************** -->
     <link name="base_footprint"/>
     <joint name="base_joint" type="fixed">
-        <origin xyz="0.0 0.0 0.0" rpy="0.0 0.0 0.0"/>
+        <origin xyz="0.0 0.0 0.1" rpy="0.0 0.0 0.0"/>
         <parent link="base_footprint"/>
         <child link="base_link"/>
@@ -21,16 +16,16 @@
             <origin xyz="0.0 0.0 0" rpy="0.0 0.0 0.0"/>
             <geometry>
-                <mesh filename="file:///$(find robot_descriptions)/urdf/chocolate_bot/meshes/base_link.dae" scale="1 1 1"/>
+                <mesh filename="file:///$(find robot_descriptions)/urdf/chocolate_bot/meshes/base_link.dae" scale="10 10 10"/>
             </geometry>
             <material name="Blue"/>
         </visual>
         <collision>
-            <origin xyz="0.0 0.0 0" rpy="0.0 0.0 0.0"/>
+            <origin xyz="0.0 0.0 0.2" rpy="0.0 0.0 1.57"/>
             <geometry>
-                <box size="0.15 0.10 0.06"/>
+                <box size="1.5 1.0 0.6"/>
             </geometry>
         </collision>
-        <xacro:box_inertia mass="1.5" length="0.15" width="0.10" height="0.06"
-                            xyz="0 0 0" rpy="0 0 0" />
+        <xacro:box_inertia mass="1.5" length="1.5" width="1.0" height="0.6"
+                            xyz="0.0 0.0 0.3" rpy="1.57 0 0.0" />
     </link>
     <gazebo reference="base_link">
@@ -38,44 +33,42 @@
     </gazebo>
 <!-- ********************** Wheel links and joints ********************** -->
-    <xacro:macro name="wheel_link" params="prefix xyz rpy">
+    <xacro:macro name="wheel_link" params="prefix xyz rpy Jrpy">
         <link name="${prefix}_wheel_link">
             <visual name="rim">
-                <origin xyz="0 0 0" rpy="0 0 0" />
+                <origin xyz="0 0 0" rpy="${rpy}" />
                 <geometry>
-                    <mesh filename="file:///$(find robot_descriptions)/urdf/chocolate_bot/meshes/wheel_rim.dae"  scale="1 1 1"/>
+                    <mesh filename="file:///$(find robot_descriptions)/urdf/chocolate_bot/meshes/wheel_rim.dae"  scale="10 10 10"/>
                 </geometry>
                 <material name="Red" />
             </visual>
-            <visual name="tyre">
+<!--             <visual name="tyre">
                 <origin xyz="0 0 0" rpy="0 0 0" />
                 <geometry>
-                    <mesh filename="file:///$(find robot_descriptions)/urdf/chocolate_bot/meshes/wheel_tyre.dae"  scale="1 1 1"/>
+                    <mesh filename="file:///$(find robot_descriptions)/urdf/chocolate_bot/meshes/wheel_tyre.dae"  scale="10 10 10"/>
                 </geometry>
                 <material name="Black" />
-            </visual>
+            </visual> -->
             <collision>
-                <origin xyz="0 0 0" rpy="0 0 0" />
+                <origin xyz="0.015 0 0" rpy="0 1.57 0" />
                 <geometry>
+                    <cylinder radius="0.15" length="0.03"/>
                 </geometry>
             </collision>
-            <!-- <xacro:cylinder_inertia mass="0.05" radius="${wheel_radius}" height="${wheel_length}"
-                                    xyz="0 0 0" rpy="${pi / 2.0} 0 0" /> -->
+            <xacro:cylinder_inertia mass="0.05" radius="0.15" height="0.03"
+                                    xyz="0.015 0 0" rpy="0 1.57 0" />
         </link>
         <joint name="base_${prefix}_wheel_joint" type="continuous">
-            <origin xyz="${xyz}" rpy="${rpy}"/>
+            <origin xyz="${xyz}" rpy="${Jrpy}"/>
             <parent link="base_link"/>
             <child link="${prefix}_wheel_link"/>
             <axis xyz="1 0.0 0.0"/>
         </joint>
-        <gazebo reference="rim">
-            <material>Gazebo/Red</material>
-        </gazebo>
-        <gazebo reference="tyre">
+        <gazebo reference="wheel_link">
             <material>Gazebo/Red</material>
         </gazebo>
     </xacro:macro>
-    <xacro:wheel_link prefix="front_right" xyz="0.05 0.05 0.005" rpy="0 0 0"/>
-    <xacro:wheel_link prefix="back_right" xyz="0.05 -0.05 0.005" rpy="0 0 0"/>
-    <xacro:wheel_link prefix="front_left" xyz="-0.05 0.05 0.005" rpy="0 0 3.14"/>
-    <xacro:wheel_link prefix="back_left" xyz="-0.05 -0.05 0.005" rpy="0 0 3.14"/>
+    <xacro:wheel_link prefix="front_right" xyz="0.5 0.5 0.05" rpy="0 0 0" Jrpy="0 0 0"/>
+    <xacro:wheel_link prefix="back_right" xyz="0.5 -0.5 0.05" rpy="0 0 0" Jrpy="0 0 0"/>
+    <xacro:wheel_link prefix="front_left" xyz="-0.5 0.5 0.05" rpy="0 0 3.014" Jrpy="0 0 0"/>
+    <xacro:wheel_link prefix="back_left" xyz="-0.5 -0.5 0.05" rpy="0 0 3.14" Jrpy="0 0 0"/>
 </robot>

File: robot_descriptions/urdf/chocolate_bot/chocolate_bot_urdf.xacro (robot description, xacro)
@@ -2,6 +2,5 @@
 <robot name="chocolate_bot" xmlns:xacro="http://www.ros.org/wiki/xacro">
     <xacro:include filename="$(find robot_descriptions)/urdf/common_parameters.xacro" />
-    <!-- <xacro:include filename="$(find robot_descriptions)/urdf/plugins/imu.xacro" />
-    <xacro:include filename="$(find robot_descriptions)/urdf/plugins/camera.xacro" /> -->
+    <xacro:include filename="$(find robot_descriptions)/urdf/plugins/skid_steer_drive.xacro" />
     <xacro:include filename="chocolate_bot_base.xacro" />
 </robot>

Commit message: added skid_steer

File: robot_descriptions/urdf/chocolate_bot/chocolate_bot_base.xacro (robot description, xacro)
@@ -3,5 +3,5 @@
     <xacro:skid_steer_drive leftFrontJoint = "base_front_left_wheel_joint" rightFrontJoint = "base_front_right_wheel_joint"
                             leftRearJoint = "base_back_left_wheel_joint" rightRearJoint = "base_back_right_wheel_joint"
-                            robotBaseFrame = "base_link" wheelDiameter = "0.165" wheelSeparation = "1" />
+                            robotBaseFrame = "base_footprint" wheelDiameter = "0.165" wheelSeparation = "1.2" />
 <!-- ********************** Base footprint link and joint ********************** -->
     <link name="base_footprint"/>
@@ -21,5 +21,5 @@
         </visual>
         <collision>
-            <origin xyz="0.0 0.0 0.2" rpy="0.0 0.0 1.57"/>
+            <origin xyz="0.0 0.0 0.3" rpy="0.0 0.0 1.57"/>
             <geometry>
                 <box size="1.5 1.0 0.6"/>
@@ -33,5 +33,5 @@
     </gazebo>
 <!-- ********************** Wheel links and joints ********************** -->
-    <xacro:macro name="wheel_link" params="prefix xyz rpy Jrpy">
+    <xacro:macro name="wheel_link" params="prefix xyz rpy Jrpy Ixyz Cxyz">
         <link name="${prefix}_wheel_link">
             <visual name="rim">
@@ -50,11 +50,11 @@
             </visual> -->
             <collision>
-                <origin xyz="0.015 0 0" rpy="0 1.57 0" />
+                <origin xyz="${Cxyz}" rpy="0 1.57 0" />
                 <geometry>
                     <cylinder radius="0.15" length="0.03"/>
                 </geometry>
             </collision>
-            <xacro:cylinder_inertia mass="0.05" radius="0.15" height="0.03"
-                                    xyz="0.015 0 0" rpy="0 1.57 0" />
+            <xacro:cylinder_inertia mass="0.05" radius="0.3" height="0.06"
+                                    xyz="${Ixyz}" rpy="0 1.57 0" />
         </link>
         <joint name="base_${prefix}_wheel_joint" type="continuous">
@@ -64,11 +64,12 @@
             <axis xyz="1 0.0 0.0"/>
         </joint>
-        <gazebo reference="wheel_link">
-            <material>Gazebo/Red</material>
+        <gazebo reference="${prefix}_wheel_link">
+            <mu1 value="1" />
+            <mu2 value="1" />
         </gazebo>
     </xacro:macro>
-    <xacro:wheel_link prefix="front_right" xyz="0.5 0.5 0.05" rpy="0 0 0" Jrpy="0 0 0"/>
-    <xacro:wheel_link prefix="back_right" xyz="0.5 -0.5 0.05" rpy="0 0 0" Jrpy="0 0 0"/>
-    <xacro:wheel_link prefix="front_left" xyz="-0.5 0.5 0.05" rpy="0 0 3.014" Jrpy="0 0 0"/>
-    <xacro:wheel_link prefix="back_left" xyz="-0.5 -0.5 0.05" rpy="0 0 3.14" Jrpy="0 0 0"/>
+    <xacro:wheel_link prefix="front_right" xyz="0.6 0.5 0.025" rpy="0 0 0" Jrpy="0 0 0" Ixyz="0.015 0 0" Cxyz="0.015 0 0"/>
+    <xacro:wheel_link prefix="back_right" xyz="0.6 -0.5 0.025" rpy="0 0 0" Jrpy="0 0 0" Ixyz="0.015 0 0" Cxyz="0.015 0 0"/>
+    <xacro:wheel_link prefix="front_left" xyz="-0.6 0.5 0.025" rpy="0 0 3.14" Jrpy="0 0 0" Ixyz="-0.015 0 0" Cxyz="-0.015 0 0"/>
+    <xacro:wheel_link prefix="back_left" xyz="-0.6 -0.5 0.025" rpy="0 0 3.14" Jrpy="0 0 0" Ixyz="-0.015 0 0" Cxyz="-0.015 0 0"/>
 </robot>

File: robot_descriptions/urdf/plugins/skid_steer_drive.xacro (robot description, xacro)
@@ -4,5 +4,5 @@
                                                     wheelDiameter wheelSeparation">
         <gazebo>
-            <plugin name="skid_steer_drive_controller" filename="libgazebo_ros_diff_drive.so">
+            <plugin name="skid_steer_drive" filename="libgazebo_ros_diff_drive.so">
                 <!-- Number of wheel pairs -->
                 <num_wheel_pairs>2</num_wheel_pairs>
@@ -19,13 +19,13 @@
                 <wheel_diameter>${wheelDiameter}</wheel_diameter>
                 <!-- limits -->
-                <max_wheel_torque>20</max_wheel_torque>
+                <max_wheel_torque>10</max_wheel_torque>
                 <max_wheel_acceleration>1.0</max_wheel_acceleration>
                 <robotBaseFrame>${robotBaseFrame}</robotBaseFrame>
                 <!-- output -->
                 <update_rate>30.0</update_rate>
-                <odometry_frame>odom</odometry_frame>
                 <publish_odom>true</publish_odom>
                 <publish_odom_tf>true</publish_odom_tf>
                 <publish_wheel_tf>true</publish_wheel_tf>
+                <odometry_frame>odom</odometry_frame>
                 <robot_base_frame>${robotBaseFrame}</robot_base_frame>
             </plugin>

Commit message: nav2

File: robot_descriptions/urdf/chocolate_bot/chocolate_bot_base.xacro (robot description, xacro)
@@ -42,11 +42,4 @@
                 <material name="Red" />
             </visual>
-<!--             <visual name="tyre">
-                <origin xyz="0 0 0" rpy="0 0 0" />
-                <geometry>
-                    <mesh filename="file:///$(find robot_descriptions)/urdf/chocolate_bot/meshes/wheel_tyre.dae"  scale="10 10 10"/>
-                </geometry>
-                <material name="Black" />
-            </visual> -->
             <collision>
                 <origin xyz="${Cxyz}" rpy="0 1.57 0" />
@@ -67,4 +60,8 @@
             <mu1 value="1" />
             <mu2 value="1" />
+            <kp value="500000.0" />
+            <kd value="10.0"/>
+            <minDepth value="0.001"/>
+            <maxVel value="1"/>
         </gazebo>
     </xacro:macro>

File: robot_descriptions/urdf/plugins/skid_steer_drive.xacro (robot description, xacro)
@@ -20,5 +20,5 @@
                 <!-- limits -->
                 <max_wheel_torque>10</max_wheel_torque>
-                <max_wheel_acceleration>1.0</max_wheel_acceleration>
+                <max_wheel_acceleration>2.0</max_wheel_acceleration>
                 <robotBaseFrame>${robotBaseFrame}</robotBaseFrame>
                 <!-- output -->
